File: esp433.sch (KiCad schematic (older format))
At the start: 35 parts, among them J1 USB_OTG, J2 CONN_01X03, Q1 MBT2222ADW1T1, SW1 SW_Push, U1 AP2127K-3.3, U2 IRM-02-5, U3 ESP-12E, U4 FT231XS

Commit message: Add rf circuit
Parts:
- added AE1: Antenna, esp433:W3127, symbol Antenna
- added C3, C8: 100n, Capacitors_SMD:C_0603, symbol C
- added C4: 220p, Capacitors_SMD:C_0603, symbol C
- added C5: 680p, Capacitors_SMD:C_0603, symbol C
- added C6, C7: 12p, Capacitors_SMD:C_0603, symbol C
- added L2: 27nH, Inductors_SMD:L_0603, symbol L
- added L3: 15nH, Inductors_SMD:L_0603, symbol L
- added R6: R_Variable, Potentiometers:Potentiometer_Trimmer_Vishay_TS53YL, symbol R_Variable
- added U3: MAX7044, TO_SOT_Packages_SMD:SOT-23-8, symbol MAX7044
- added Y1: Crystal, Crystals:Crystal_HC49-U_Vertical, symbol Crystal
- SW1: footprint Buttons_Switches_SMD:SW_SPST_PTS645 -> Buttons_Switches_SMD:SW_SPST_B3U-1000P; Vendorpart CKN9112CT-ND -> SW1020CT-ND
- renumbered C7 to C1, C2 to C10, C3 to C11, C4 to C12, C5 to C13, C6 to C14, C8 to C2, C1 to C9, R9 to R10, R10 to R11, R6 to R7, R7 to R9, U2 to U1, U1 to U2, U3 to U4, U4 to U5
Connections:
- net +3V3: now also C8.1, R6.1, U3.7 (VDD)
- net GND: now also C3.2, C4.2, C5.2, C6.2, C7.2, C8.2, U3.2 (GND), U3.3 (PAGND)
- net RF_MOD: now also U3.6 (DATA)
- net RF_CLK: now reaches U4.5 (GPIO14)
- net RF_CLK: now also U3.5 (CLKOUT)
- new net: U3.1 (XTAL1), Y1.1
- new net: C7.1, L2.2, L3.1, U3.4 (PAOUT)
- new net: U3.8 (XTAL2), Y1.2
- new net: C3.1, C4.1, C5.1, L2.1, R6.2
- new net: AE1.1 (A), C6.1, L3.2
- no-connect marks 21 -> 20
Other:
- moved on the sheet: J2, R9, U4

Commit message: Rearrange filtering according to datasheet
Connections:
- net +3V3: now also C3.1
- net at C4.1, C5.1, L2.1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: no longer C3.1
Changed lines of the file:
@@
 $EndComp
-Wire Wire Line
-	7550 3000 8500 3000
 Wire Wire Line
 	8500 2900 8500 3250
@@
 	8500 2600 8500 2500
 Connection ~ 8150 3000
-Connection ~ 7850 3000
+Wire Wire Line
+	7850 3000 8500 3000
+Wire Wire Line
+	7550 3000 7550 2550
+Wire Wire Line
+	7550 2550 8500 2550
+Connection ~ 8500 2550
 $EndSCHEMATC

Commit message: Rework to fix oscillator and antenna circuit
Parts:
- added C15, C16: 12p, Capacitors_SMD:C_0603, symbol C
- added C17: 15p, Capacitors_SMD:C_0603, symbol C
Connections:
- net at U3.1 (XTAL1): now also C15.2; no longer Y1.1
- net at L2.2, U3.4 (PAOUT): now also C17.1; no longer C7.1, L3.1
- net at U3.8 (XTAL2): now also C16.1; no longer Y1.2
- new net: C15.1, Y1.1
- new net: C16.2, Y1.2
- new net: C17.2, C7.1, L3.1

Commit message: Fix footprint for D1
Parts:
- D1: footprint Diodes_SMD:D_0603 -> Diodes_SMD:D_SOD-123F
Changed lines of the file:
@@
 $EndComp
 $Comp
-L GND #PWR9
+L GND #PWR01
 U 1 1 5A6C1DE7
 P 4850 2650
-F 0 "#PWR9" H 4850 2400 50  0001 C CNN
+F 0 "#PWR01" H 4850 2400 50  0001 C CNN
 F 1 "GND" H 4850 2500 50  0000 C CNN
 F 2 "" H 4850 2650 50  0001 C CNN
@@
 $EndComp
 $Comp
-L +3V3 #PWR5
+L +3V3 #PWR02
 U 1 1 5A6C1E2B
 P 5500 1650
-F 0 "#PWR5" H 5500 1500 50  0001 C CNN
+F 0 "#PWR02" H 5500 1500 50  0001 C CNN
 F 1 "+3V3" H 5500 1790 50  0000 C CNN
 F 2 "" H 5500 1650 50  0001 C CNN
@@
 $EndComp
 $Comp
-L +5V #PWR4
+L +5V #PWR03
 U 1 1 5A6C1E6F
 P 4350 1650
-F 0 "#PWR4" H 4350 1500 50  0001 C CNN
+F 0 "#PWR03" H 4350 1500 50  0001 C CNN
 F 1 "+5V" H 4350 1790 50  0000 C CNN
 F 2 "" H 4350 1650 50  0001 C CNN
@@
 $EndComp
 $Comp
-L +3V3 #PWR1
+L +3V3 #PWR04
 U 1 1 5A6C1EEB
 P 9550 1350
-F 0 "#PWR1" H 9550 1200 50  0001 C CNN
+F 0 "#PWR04" H 9550 1200 50  0001 C CNN
 F 1 "+3V3" H 9550 1490 50  0000 C CNN
 F 2 "" H 9550 1350 50  0001 C CNN
@@
 $EndComp
 $Comp
-L +3V3 #PWR2
+L +3V3 #PWR05
 U 1 1 5A6C1F26
 P 10000 1350
-F 0 "#PWR2" H 10000 1200 50  0001 C CNN
+F 0 "#PWR05" H 10000 1200 50  0001 C CNN
 F 1 "+3V3" H 10000 1490 50  0000 C CNN
 F 2 "" H 10000 1350 50  0001 C CNN
@@
 GPIO0
 $Comp
-L GND #PWR29
+L GND #PWR06
 U 1 1 5A6D5837
 P 9150 5550
-F 0 "#PWR29" H 9150 5300 50  0001 C CNN
+F 0 "#PWR06" H 9150 5300 50  0001 C CNN
 F 1 "GND" H 9150 5400 50  0000 C CNN
 F 2 "" H 9150 5550 50  0001 C CNN
@@
 $EndComp
 $Comp
-L +3V3 #PWR28
+L +3V3 #PWR07
 U 1 1 5A6D58FF
 P 7600 5400
-F 0 "#PWR28" H 7600 5250 50  0001 C CNN
+F 0 "#PWR07" H 7600 5250 50  0001 C CNN
 F 1 "+3V3" H 7600 5540 50  0000 C CNN
 F 2 "" H 7600 5400 50  0001 C CNN
@@
 GPIO15
 $Comp
-L GND #PWR7
+L GND #PWR08
 U 1 1 5A6D5ED0
 P 10400 2050
-F 0 "#PWR7" H 10400 1800 50  0001 C CNN
+F 0 "#PWR08" H 10400 1800 50  0001 C CNN
 F 1 "GND" H 10400 1900 50  0000 C CNN
 F 2 "" H 10400 2050 50  0001 C CNN
@@
 $EndComp
 $Comp
-L +3V3 #PWR15
+L +3V3 #PWR09
 U 1 1 5A6D623C
 P 3850 3450
-F 0 "#PWR15" H 3850 3300 50  0001 C CNN
+F 0 "#PWR09" H 3850 3300 50  0001 C CNN
 F 1 "+3V3" H 3850 3590 50  0000 C CNN
 F 2 "" H 3850 3450 50  0001 C CNN
@@
 $EndComp
 $Comp
-L GND #PWR24
+L GND #PWR010
 U 1 1 5A6D62B4
 P 6050 4700
-F 0 "#PWR24" H 6050 4450 50  0001 C CNN
+F 0 "#PWR010" H 6050 4450 50  0001 C CNN
 F 1 "GND" H 6050 4550 50  0000 C CNN
 F 2 "" H 6050 4700 50  0001 C CNN
@@
 $EndComp
 $Comp
-L +5V #PWR25
+L +5V #PWR011
 U 1 1 5A6D6578
 P 3000 5050
-F 0 "#PWR25" H 3000 4900 50  0001 C CNN
+F 0 "#PWR011" H 3000 4900 50  0001 C CNN
 F 1 "+5V" H 3000 5190 50  0000 C CNN
 F 2 "" H 3000 5050 50  0001 C CNN
@@
 $EndComp
 $Comp
-L GND #PWR33
+L GND #PWR012
 U 1 1 5A6D65B9
 P 3000 7200
-F 0 "#PWR33" H 3000 6950 50  0001 C CNN
+F 0 "#PWR012" H 3000 6950 50  0001 C CNN
 F 1 "GND" H 3000 7050 50  0000 C CNN
 F 2 "" H 3000 7200 50  0001 C CNN
@@
 $EndComp
 $Comp
-L GND #PWR34
+L GND #PWR013
 U 1 1 5A6D65FA
 P 3200 7200
-F 0 "#PWR34" H 3200 6950 50  0001 C CNN
+F 0 "#PWR013" H 3200 6950 50  0001 C CNN
 F 1 "GND" H 3200 7050 50  0000 C CNN
 F 2 "" H 3200 7200 50  0001 C CNN
@@
 $EndComp
 $Comp
-L +5V #PWR11
+L +5V #PWR014
 U 1 1 5A6D6D35
 P 2650 3100
-F 0 "#PWR11" H 2650 2950 50  0001 C CNN
+F 0 "#PWR014" H 2650 2950 50  0001 C CNN
 F 1 "+5V" H 2650 3240 50  0000 C CNN
 F 2 "" H 2650 3100 50  0001 C CNN
@@
 $EndComp
 $Comp
-L GND #PWR16
+L GND #PWR015
 U 1 1 5A6D6EA9
 P 1550 4050
-F 0 "#PWR16" H 1550 3800 50  0001 C CNN
+F 0 "#PWR015" H 1550 3800 50  0001 C CNN
 F 1 "GND" H 1550 3900 50  0000 C CNN
 F 2 "" H 1550 4050 50  0001 C CNN
@@
 F 0 "D1" H 2850 1750 50  0000 C CNN
 F 1 "D" H 2850 1550 50  0000 C CNN
-F 2 "Diodes_SMD:D_0603" H 2850 1650 50  0001 C CNN
+F 2 "Diodes_SMD:D_SOD-123F" H 2850 1650 50  0001 C CNN
 F 3 "" H 2850 1650 50  0001 C CNN
 F 4 "MBR120VLSFT3GOSCT-ND" H 2850 1650 60  0000 C CNN "Vendorpart"
@@
 $EndComp
 $Comp
-L GND #PWR6
+L GND #PWR016
 U 1 1 5A6D85B9
 P 2650 1850
-F 0 "#PWR6" H 2650 1600 50  0001 C CNN
+F 0 "#PWR016" H 2650 1600 50  0001 C CNN
 F 1 "GND" H 2650 1700 50  0000 C CNN
 F 2 "" H 2650 1850 50  0001 C CNN
@@
 $EndComp
 $Comp
-L +5V #PWR3
+L +5V #PWR017
 U 1 1 5A6D867B
 P 3200 1500
-F 0 "#PWR3" H 3200 1350 50  0001 C CNN
+F 0 "#PWR017" H 3200 1350 50  0001 C CNN
 F 1 "+5V" H 3200 1640 50  0000 C CNN
 F 2 "" H 3200 1500 50  0001 C CNN
@@
 $EndComp
 $Comp
-L +3V3 #PWR30
+L +3V3 #PWR018
 U 1 1 5A6D9A1C
 P 5900 5700
-F 0 "#PWR30" H 5900 5550 50  0001 C CNN
+F 0 "#PWR018" H 5900 5550 50  0001 C CNN
 F 1 "+3V3" H 5900 5840 50  0000 C CNN
 F 2 "" H 5900 5700 50  0001 C CNN
@@
 $EndComp
 $Comp
-L +3V3 #PWR23
+L +3V3 #PWR019
 U 1 1 5A6DA721
 P 9250 4600
-F 0 "#PWR23" H 9250 4450 50  0001 C CNN
+F 0 "#PWR019" H 9250 4450 50  0001 C CNN
 F 1 "+3V3" H 9250 4740 50  0000 C CNN
 F 2 "" H 9250 4600 50  0001 C CNN
@@
 $EndComp
 $Comp
-L GND #PWR27
+L GND #PWR020
 U 1 1 5A6DA77A
 P 9250 5100
-F 0 "#PWR27" H 9250 4850 50  0001 C CNN
+F 0 "#PWR020" H 9250 4850 50  0001 C CNN
 F 1 "GND" H 9250 4950 50  0000 C CNN
 F 2 "" H 9250 5100 50  0001 C CNN
@@
 $EndComp
 $Comp
-L GND #PWR22
+L GND #PWR021
 U 1 1 5A6DD0A2
 P 2650 4400
-F 0 "#PWR22" H 2650 4150 50  0001 C CNN
+F 0 "#PWR021" H 2650 4150 50  0001 C CNN
 F 1 "GND" H 2650 4250 50  0000 C CNN
 F 2 "" H 2650 4400 50  0001 C CNN
@@
 $EndComp
 $Comp
-L GND #PWR21
+L GND #PWR022
 U 1 1 5A6DD462
 P 2000 4400
-F 0 "#PWR21" H 2000 4150 50  0001 C CNN
+F 0 "#PWR022" H 2000 4150 50  0001 C CNN
 F 1 "GND" H 2000 4250 50  0000 C CNN
 F 2 "" H 2000 4400 50  0001 C CNN
@@
 $EndComp
 $Comp
-L +5V #PWR31
+L +5V #PWR023
 U 1 1 5A6DE01F
 P 1650 6550
-F 0 "#PWR31" H 1650 6400 50  0001 C CNN
+F 0 "#PWR023" H 1650 6400 50  0001 C CNN
 F 1 "+5V" H 1650 6690 50  0000 C CNN
 F 2 "" H 1650 6550 50  0001 C CNN
@@
 $EndComp
 $Comp
-L GND #PWR32
+L GND #PWR024
 U 1 1 5A6DE1A7
 P 1650 7150
-F 0 "#PWR32" H 1650 6900 50  0001 C CNN
+F 0 "#PWR024" H 1650 6900 50  0001 C CNN
 F 1 "GND" H 1650 7000 50  0000 C CNN
 F 2 "" H 1650 7150 50  0001 C CNN
@@
 AC-N
 $Comp
-L +3V3 #PWR26
+L +3V3 #PWR025
 U 1 1 5A6D6537
 P 3200 5050
-F 0 "#PWR26" H 3200 4900 50  0001 C CNN
+F 0 "#PWR025" H 3200 4900 50  0001 C CNN
 F 1 "+3V3" H 3200 5190 50  0000 C CNN
 F 2 "" H 3200 5050 50  0001 C CNN
@@
 $EndComp
 $Comp
-L GND #PWR20
+L GND #PWR026
 U 1 1 5A766445
 P 10350 4150
-F 0 "#PWR20" H 10350 3900 50  0001 C CNN
+F 0 "#PWR026" H 10350 3900 50  0001 C CNN
 F 1 "GND" H 10350 4000 50  0000 C CNN
 F 2 "" H 10350 4150 50  0001 C CNN
@@
 $EndComp
 $Comp
-L +3V3 #PWR10
+L +3V3 #PWR027
 U 1 1 5A7665C1
 P 10350 2800
-F 0 "#PWR10" H 10350 2650 50  0001 C CNN
+F 0 "#PWR027" H 10350 2650 50  0001 C CNN
 F 1 "+3V3" H 10350 2940 50  0000 C CNN
 F 2 "" H 10350 2800 50  0001 C CNN
@@
 $EndComp
 $Comp
-L GND #PWR19
+L GND #PWR028
 U 1 1 5A7669B1
 P 8750 4100
-F 0 "#PWR19" H 8750 3850 50  0001 C CNN
+F 0 "#PWR028" H 8750 3850 50  0001 C CNN
 F 1 "GND" H 8750 3950 50  0000 C CNN
 F 2 "" H 8750 4100 50  0001 C CNN
@@
 $EndComp
 $Comp
-L +3V3 #PWR8
+L +3V3 #PWR029
 U 1 1 5A767193
 P 8500 2500
-F 0 "#PWR8" H 8500 2350 50  0001 C CNN
+F 0 "#PWR029" H 8500 2350 50  0001 C CNN
 F 1 "+3V3" H 8500 2640 50  0000 C CNN
 F 2 "" H 8500 2500 50  0001 C CNN
@@
 $EndComp
 $Comp
-L GND #PWR18
+L GND #PWR030
 U 1 1 5A767EA9
 P 8000 4100
-F 0 "#PWR18" H 8000 3850 50  0001 C CNN
+F 0 "#PWR030" H 8000 3850 50  0001 C CNN
 F 1 "GND" H 8000 3950 50  0000 C CNN
 F 2 "" H 8000 4100 50  0001 C CNN
@@
 $EndComp
 $Comp
-L GND #PWR17
+L GND #PWR031
 U 1 1 5A767F41
 P 7350 4100
-F 0 "#PWR17" H 7350 3850 50  0001 C CNN
+F 0 "#PWR031" H 7350 3850 50  0001 C CNN
 F 1 "GND" H 7350 3950 50  0000 C CNN
 F 2 "" H 7350 4100 50  0001 C CNN
@@
 RF_CLK
 $Comp
-L GND #PWR14
+L GND #PWR032
 U 1 1 5A769625
 P 8150 3300
-F 0 "#PWR14" H 8150 3050 50  0001 C CNN
+F 0 "#PWR032" H 8150 3050 50  0001 C CNN
 F 1 "GND" H 8150 3150 50  0000 C CNN
 F 2 "" H 8150 3300 50  0001 C CNN
@@
 $EndComp
 $Comp
-L GND #PWR13
+L GND #PWR033
 U 1 1 5A7696BD
 P 7850 3300
-F 0 "#PWR13" H 7850 3050 50  0001 C CNN
+F 0 "#PWR033" H 7850 3050 50  0001 C CNN
 F 1 "GND" H 7850 3150 50  0000 C CNN
 F 2 "" H 7850 3300 50  0001 C CNN
@@
 $EndComp
 $Comp
-L GND #PWR12
+L GND #PWR034
 U 1 1 5A769755
 P 7550 3300
-F 0 "#PWR12" H 7550 3050 50  0001 C CNN
+F 0 "#PWR034" H 7550 3050 50  0001 C CNN
 F 1 "GND" H 7550 3150 50  0000 C CNN
 F 2 "" H 7550 3300 50  0001 C CNN

Commit message: Add some dnp footprints for additional oscillator parallel capacitance
Parts:
- added C18, C19: DNP, Capacitors_SMD:C_0603, symbol C
Connections:
- net GND: now also C18.1, C19.1
- net at C15.2, U3.1 (XTAL1): now also C18.2
- net at C16.1, U3.8 (XTAL2): now also C19.2
Changed lines of the file:
@@
 $EndComp
 $Comp
-L GND #PWR01
+L GND #PWR9
 U 1 1 5A6C1DE7
 P 4850 2650
-F 0 "#PWR01" H 4850 2400 50  0001 C CNN
+F 0 "#PWR9" H 4850 2400 50  0001 C CNN
 F 1 "GND" H 4850 2500 50  0000 C CNN
 F 2 "" H 4850 2650 50  0001 C CNN
@@
 $EndComp
 $Comp
-L +3V3 #PWR02
+L +3V3 #PWR5
 U 1 1 5A6C1E2B
 P 5500 1650
-F 0 "#PWR02" H 5500 1500 50  0001 C CNN
+F 0 "#PWR5" H 5500 1500 50  0001 C CNN
 F 1 "+3V3" H 5500 1790 50  0000 C CNN
 F 2 "" H 5500 1650 50  0001 C CNN
@@
 $EndComp
 $Comp
-L +5V #PWR03
+L +5V #PWR4
 U 1 1 5A6C1E6F
 P 4350 1650
-F 0 "#PWR03" H 4350 1500 50  0001 C CNN
+F 0 "#PWR4" H 4350 1500 50  0001 C CNN
 F 1 "+5V" H 4350 1790 50  0000 C CNN
 F 2 "" H 4350 1650 50  0001 C CNN
@@
 $EndComp
 $Comp
-L +3V3 #PWR04
+L +3V3 #PWR1
 U 1 1 5A6C1EEB
 P 9550 1350
-F 0 "#PWR04" H 9550 1200 50  0001 C CNN
+F 0 "#PWR1" H 9550 1200 50  0001 C CNN
 F 1 "+3V3" H 9550 1490 50  0000 C CNN
 F 2 "" H 9550 1350 50  0001 C CNN
@@
 $EndComp
 $Comp
-L +3V3 #PWR05
+L +3V3 #PWR2
 U 1 1 5A6C1F26
 P 10000 1350
-F 0 "#PWR05" H 10000 1200 50  0001 C CNN
+F 0 "#PWR2" H 10000 1200 50  0001 C CNN
 F 1 "+3V3" H 10000 1490 50  0000 C CNN
 F 2 "" H 10000 1350 50  0001 C CNN
@@
 GPIO0
 $Comp
-L GND #PWR06
+L GND #PWR31
 U 1 1 5A6D5837
 P 9150 5550
-F 0 "#PWR06" H 9150 5300 50  0001 C CNN
+F 0 "#PWR31" H 9150 5300 50  0001 C CNN
 F 1 "GND" H 9150 5400 50  0000 C CNN
 F 2 "" H 9150 5550 50  0001 C CNN
@@
 $EndComp
 $Comp
-L +3V3 #PWR07
+L +3V3 #PWR30
 U 1 1 5A6D58FF
 P 7600 5400
-F 0 "#PWR07" H 7600 5250 50  0001 C CNN
+F 0 "#PWR30" H 7600 5250 50  0001 C CNN
 F 1 "+3V3" H 7600 5540 50  0000 C CNN
 F 2 "" H 7600 5400 50  0001 C CNN
@@
 GPIO15
 $Comp
-L GND #PWR08
+L GND #PWR7
 U 1 1 5A6D5ED0
 P 10400 2050
-F 0 "#PWR08" H 10400 1800 50  0001 C CNN
+F 0 "#PWR7" H 10400 1800 50  0001 C CNN
 F 1 "GND" H 10400 1900 50  0000 C CNN
 F 2 "" H 10400 2050 50  0001 C CNN
@@
 $EndComp
 $Comp
-L +3V3 #PWR09
+L +3V3 #PWR17
 U 1 1 5A6D623C
 P 3850 3450
-F 0 "#PWR09" H 3850 3300 50  0001 C CNN
+F 0 "#PWR17" H 3850 3300 50  0001 C CNN
 F 1 "+3V3" H 3850 3590 50  0000 C CNN
 F 2 "" H 3850 3450 50  0001 C CNN
@@
 $EndComp
 $Comp
-L GND #PWR010
+L GND #PWR26
 U 1 1 5A6D62B4
 P 6050 4700
-F 0 "#PWR010" H 6050 4450 50  0001 C CNN
+F 0 "#PWR26" H 6050 4450 50  0001 C CNN
 F 1 "GND" H 6050 4550 50  0000 C CNN
 F 2 "" H 6050 4700 50  0001 C CNN
@@
 $EndComp
 $Comp
-L +5V #PWR011
+L +5V #PWR27
 U 1 1 5A6D6578
 P 3000 5050
-F 0 "#PWR011" H 3000 4900 50  0001 C CNN
+F 0 "#PWR27" H 3000 4900 50  0001 C CNN
 F 1 "+5V" H 3000 5190 50  0000 C CNN
 F 2 "" H 3000 5050 50  0001 C CNN
@@
 $EndComp
 $Comp
-L GND #PWR012
+L GND #PWR35
 U 1 1 5A6D65B9
 P 3000 7200
-F 0 "#PWR012" H 3000 6950 50  0001 C CNN
+F 0 "#PWR35" H 3000 6950 50  0001 C CNN
 F 1 "GND" H 3000 7050 50  0000 C CNN
 F 2 "" H 3000 7200 50  0001 C CNN
@@
 $EndComp
 $Comp
-L GND #PWR013
+L GND #PWR36
 U 1 1 5A6D65FA
 P 3200 7200
-F 0 "#PWR013" H 3200 6950 50  0001 C CNN
+F 0 "#PWR36" H 3200 6950 50  0001 C CNN
 F 1 "GND" H 3200 7050 50  0000 C CNN
 F 2 "" H 3200 7200 50  0001 C CNN
@@
 $EndComp
 $Comp
-L +5V #PWR014
+L +5V #PWR11
 U 1 1 5A6D6D35
 P 2650 3100
-F 0 "#PWR014" H 2650 2950 50  0001 C CNN
+F 0 "#PWR11" H 2650 2950 50  0001 C CNN
 F 1 "+5V" H 2650 3240 50  0000 C CNN
 F 2 "" H 2650 3100 50  0001 C CNN
@@
 $EndComp
 $Comp
-L GND #PWR015
+L GND #PWR18
 U 1 1 5A6D6EA9
 P 1550 4050
-F 0 "#PWR015" H 1550 3800 50  0001 C CNN
+F 0 "#PWR18" H 1550 3800 50  0001 C CNN
 F 1 "GND" H 1550 3900 50  0000 C CNN
 F 2 "" H 1550 4050 50  0001 C CNN
@@
 $EndComp
 $Comp
-L GND #PWR016
+L GND #PWR6
 U 1 1 5A6D85B9
 P 2650 1850
-F 0 "#PWR016" H 2650 1600 50  0001 C CNN
+F 0 "#PWR6" H 2650 1600 50  0001 C CNN
 F 1 "GND" H 2650 1700 50  0000 C CNN
 F 2 "" H 2650 1850 50  0001 C CNN
@@
 $EndComp
 $Comp
-L +5V #PWR017
+L +5V #PWR3
 U 1 1 5A6D867B
 P 3200 1500
-F 0 "#PWR017" H 3200 1350 50  0001 C CNN
+F 0 "#PWR3" H 3200 1350 50  0001 C CNN
 F 1 "+5V" H 3200 1640 50  0000 C CNN
 F 2 "" H 3200 1500 50  0001 C CNN
@@
 $EndComp
 $Comp
-L +3V3 #PWR018
+L +3V3 #PWR32
 U 1 1 5A6D9A1C
 P 5900 5700
-F 0 "#PWR018" H 5900 5550 50  0001 C CNN
+F 0 "#PWR32" H 5900 5550 50  0001 C CNN
 F 1 "+3V3" H 5900 5840 50  0000 C CNN
 F 2 "" H 5900 5700 50  0001 C CNN
@@
 $EndComp
 $Comp
-L +3V3 #PWR019
+L +3V3 #PWR25
 U 1 1 5A6DA721
 P 9250 4600
-F 0 "#PWR019" H 9250 4450 50  0001 C CNN
+F 0 "#PWR25" H 9250 4450 50  0001 C CNN
 F 1 "+3V3" H 9250 4740 50  0000 C CNN
 F 2 "" H 9250 4600 50  0001 C CNN
@@
 $EndComp
 $Comp
-L GND #PWR020
+L GND #PWR29
 U 1 1 5A6DA77A
 P 9250 5100
-F 0 "#PWR020" H 9250 4850 50  0001 C CNN
+F 0 "#PWR29" H 9250 4850 50  0001 C CNN
 F 1 "GND" H 9250 4950 50  0000 C CNN
 F 2 "" H 9250 5100 50  0001 C CNN
@@
 $EndComp
 $Comp
-L GND #PWR021
+L GND #PWR24
 U 1 1 5A6DD0A2
 P 2650 4400
-F 0 "#PWR021" H 2650 4150 50  0001 C CNN
+F 0 "#PWR24" H 2650 4150 50  0001 C CNN
 F 1 "GND" H 2650 4250 50  0000 C CNN
 F 2 "" H 2650 4400 50  0001 C CNN
@@
 $EndComp
 $Comp
-L GND #PWR022
+L GND #PWR23
 U 1 1 5A6DD462
 P 2000 4400
-F 0 "#PWR022" H 2000 4150 50  0001 C CNN
+F 0 "#PWR23" H 2000 4150 50  0001 C CNN
 F 1 "GND" H 2000 4250 50  0000 C CNN
 F 2 "" H 2000 4400 50  0001 C CNN
@@
 $EndComp
 $Comp
-L +5V #PWR023
+L +5V #PWR33
 U 1 1 5A6DE01F
 P 1650 6550
-F 0 "#PWR023" H 1650 6400 50  0001 C CNN
+F 0 "#PWR33" H 1650 6400 50  0001 C CNN
 F 1 "+5V" H 1650 6690 50  0000 C CNN
 F 2 "" H 1650 6550 50  0001 C CNN
@@
 $EndComp
 $Comp
-L GND #PWR024
+L GND #PWR34
 U 1 1 5A6DE1A7
 P 1650 7150
-F 0 "#PWR024" H 1650 6900 50  0001 C CNN
+F 0 "#PWR34" H 1650 6900 50  0001 C CNN
 F 1 "GND" H 1650 7000 50  0000 C CNN
 F 2 "" H 1650 7150 50  0001 C CNN
@@
 AC-N
 $Comp
-L +3V3 #PWR025
+L +3V3 #PWR28
 U 1 1 5A6D6537
 P 3200 5050
-F 0 "#PWR025" H 3200 4900 50  0001 C CNN
+F 0 "#PWR28" H 3200 4900 50  0001 C CNN
 F 1 "+3V3" H 3200 5190 50  0000 C CNN
 F 2 "" H 3200 5050 50  0001 C CNN
@@
 $EndComp
 $Comp
-L GND #PWR026
+L GND #PWR22
 U 1 1 5A766445
 P 10350 4150
-F 0 "#PWR026" H 10350 3900 50  0001 C CNN
+F 0 "#PWR22" H 10350 3900 50  0001 C CNN
 F 1 "GND" H 10350 4000 50  0000 C CNN
 F 2 "" H 10350 4150 50  0001 C CNN
@@
 $EndComp
 $Comp
-L +3V3 #PWR027
+L +3V3 #PWR10
 U 1 1 5A7665C1
 P 10350 2800
-F 0 "#PWR027" H 10350 2650 50  0001 C CNN
+F 0 "#PWR10" H 10350 2650 50  0001 C CNN
 F 1 "+3V3" H 10350 2940 50  0000 C CNN
 F 2 "" H 10350 2800 50  0001 C CNN
@@
 $EndComp
 $Comp
-L GND #PWR028
+L GND #PWR21
 U 1 1 5A7669B1
 P 8750 4100
-F 0 "#PWR028" H 8750 3850 50  0001 C CNN
+F 0 "#PWR21" H 8750 3850 50  0001 C CNN
 F 1 "GND" H 8750 3950 50  0000 C CNN
 F 2 "" H 8750 4100 50  0001 C CNN
@@
 $EndComp
 $Comp
-L +3V3 #PWR029
+L +3V3 #PWR8
 U 1 1 5A767193
 P 8500 2500
-F 0 "#PWR029" H 8500 2350 50  0001 C CNN
+F 0 "#PWR8" H 8500 2350 50  0001 C CNN
 F 1 "+3V3" H 8500 2640 50  0000 C CNN
 F 2 "" H 8500 2500 50  0001 C CNN
@@
 $EndComp
 $Comp
-L GND #PWR030
+L GND #PWR20
 U 1 1 5A767EA9
 P 8000 4100
-F 0 "#PWR030" H 8000 3850 50  0001 C CNN
+F 0 "#PWR20" H 8000 3850 50  0001 C CNN
 F 1 "GND" H 8000 3950 50  0000 C CNN
 F 2 "" H 8000 4100 50  0001 C CNN
@@
 $EndComp
 $Comp
-L GND #PWR031
+L GND #PWR19
 U 1 1 5A767F41
 P 7350 4100
-F 0 "#PWR031" H 7350 3850 50  0001 C CNN
+F 0 "#PWR19" H 7350 3850 50  0001 C CNN
 F 1 "GND" H 7350 3950 50  0000 C CNN
 F 2 "" H 7350 4100 50  0001 C CNN
@@
 RF_CLK
 $Comp
-L GND #PWR032
+L GND #PWR16
 U 1 1 5A769625
 P 8150 3300
-F 0 "#PWR032" H 8150 3050 50  0001 C CNN
+F 0 "#PWR16" H 8150 3050 50  0001 C CNN
 F 1 "GND" H 8150 3150 50  0000 C CNN
 F 2 "" H 8150 3300 50  0001 C CNN
@@
 $EndComp
 $Comp
-L GND #PWR033
+L GND #PWR15
 U 1 1 5A7696BD
 P 7850 3300
-F 0 "#PWR033" H 7850 3050 50  0001 C CNN
+F 0 "#PWR15" H 7850 3050 50  0001 C CNN
 F 1 "GND" H 7850 3150 50  0000 C CNN
 F 2 "" H 7850 3300 50  0001 C CNN
@@
 $EndComp
 $Comp
-L GND #PWR034
+L GND #PWR14
 U 1 1 5A769755
 P 7550 3300
-F 0 "#PWR034" H 7550 3050 50  0001 C CNN
+F 0 "#PWR14" H 7550 3050 50  0001 C CNN
 F 1 "GND" H 7550 3150 50  0000 C CNN
 F 2 "" H 7550 3300 50  0001 C CNN
@@
 	8400 3700 9000 3700
 Wire Wire Line
-	8950 2900 9000 2900
+	8750 2900 9000 2900
 Wire Wire Line
 	9300 2900 9450 2900
@@
 	9750 2900 9900 2900
 Wire Wire Line
-	10200 2900 10250 2900
+	10200 2900 10600 2900
 $Comp
 L C C15
@@
 	0    1    1    0
 $EndComp
+$Comp
+L C C18
+U 1 1 5A91A9F0
+P 8750 3050
+F 0 "C18" H 8775 3150 50  0000 L CNN
+F 1 "DNP" H 8775 2950 50  0000 L CNN
+F 2 "Capacitors_SMD:C_0603" H 8788 2900 50  0001 C CNN
+F 3 "" H 8750 3050 50  0001 C CNN
+	1    8750 3050
+	-1   0    0    1
+$EndComp
+$Comp
+L C C19
+U 1 1 5A91AAB2
+P 10600 3050
+F 0 "C19" H 10625 3150 50  0000 L CNN
+F 1 "DNP" H 10625 2950 50  0000 L CNN
+F 2 "Capacitors_SMD:C_0603" H 10638 2900 50  0001 C CNN
+F 3 "" H 10600 3050 50  0001 C CNN
+	1    10600 3050
+	-1   0    0    1
+$EndComp
+Connection ~ 8950 2900
+Connection ~ 10250 2900
+$Comp
+L GND #PWR12
+U 1 1 5A91ADD1
+P 8750 3200
+F 0 "#PWR12" H 8750 2950 50  0001 C CNN
+F 1 "GND" H 8750 3050 50  0000 C CNN
+F 2 "" H 8750 3200 50  0001 C CNN
+F 3 "" H 8750 3200 50  0001 C CNN
+	1    8750 3200
+	1    0    0    -1
+$EndComp
+$Comp
+L GND #PWR13
+U 1 1 5A91AE7B
+P 10600 3200
+F 0 "#PWR13" H 10600 2950 50  0001 C CNN
+F 1 "GND" H 10600 3050 50  0000 C CNN
+F 2 "" H 10600 3200 50  0001 C CNN
+F 3 "" H 10600 3200 50  0001 C CNN
+	1    10600 3200
+	1    0    0    -1
+$EndComp
 $EndSCHEMATC
